File: Arduino_Heated_Seats_Controller.brd (EAGLE design)
At the start: 35 x 35 mm, 24 parts, among them U1 ATMEGA328P-AU, U2 UA78M05, U3 TPL7407L, U4 A2982

Commit message: Tweaking silkscreen.
Parts:
- moved U$1 3.07 mm to (23.0, 14.4)
Other:
- board text added: "ApHSC Rev. 4b"
- board text removed: "Arduino Powered Heated Seat Controller Rev. 4b"
Changed lines of the file:
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@@
 <layer number="37" name="tTest" color="7" fill="1" visible="no" active="yes"/>
 <layer number="38" name="bTest" color="7" fill="1" visible="no" active="yes"/>
-<layer number="39" name="tKeepout" color="4" fill="11" visible="yes" active="yes"/>
-<layer number="40" name="bKeepout" color="1" fill="11" visible="yes" active="yes"/>
+<layer number="39" name="tKeepout" color="4" fill="11" visible="no" active="yes"/>
+<layer number="40" name="bKeepout" color="1" fill="11" visible="no" active="yes"/>
 <layer number="41" name="tRestrict" color="4" fill="10" visible="no" active="yes"/>
 <layer number="42" name="bRestrict" color="1" fill="10" visible="no" active="yes"/>
@@
 <wire x1="24.6888" y1="29.7688" x2="22.1488" y2="29.7688" width="0.254" layer="25"/>
 <wire x1="22.1488" y1="29.7688" x2="19.6088" y2="29.7688" width="0.254" layer="25"/>
-<text x="13.6017" y="12.0777" size="0.8128" layer="22" rot="MR0" align="bottom-center">Arduino Powered Heated Seat Controller
-Rev. 4b</text>
-<text x="8.2677" y="10.9347" size="0.6096" layer="22" ratio="10" rot="MR180">https://goo.gl/t2CsID</text>
+<text x="15.7607" y="12.5857" size="0.8128" layer="22" rot="MR0" align="bottom-center">ApHSC Rev. 4b</text>
+<text x="10.8077" y="10.3632" size="0.6096" layer="22" ratio="10" rot="MR180">https://goo.gl/t2CsID</text>
 <hole x="2.5" y="2.5" drill="1.5"/>
 <hole x="2.5" y="32.5" drill="1.5"/>
@@
 <elements>
 <element name="BTN-IN" library="SparkFun-Connectors" package="1X02" value="" x="7.5819" y="32.2072" smashed="yes" rot="MR180">
-<attribute name="NAME" x="6.8707" y="30.3784" size="0.8128" layer="26" ratio="10" rot="MR180"/>
+<attribute name="NAME" x="6.7437" y="34.5694" size="0.8128" layer="26" ratio="10" rot="MR180"/>
 <attribute name="VALUE" x="6.3119" y="35.3822" size="1.27" layer="28" rot="MR180"/>
 </element>
@@
 </element>
 <element name="PWR/H" library="SparkFun-Connectors" package="1X03" value="" x="20.8788" y="31.9278" smashed="yes" rot="MR180">
-<attribute name="NAME" x="21.4376" y="30.099" size="0.8128" layer="26" ratio="10" rot="MR180"/>
+<attribute name="NAME" x="21.5646" y="34.29" size="0.8128" layer="26" ratio="10" rot="MR180"/>
 <attribute name="VALUE" x="19.6088" y="35.1028" size="1.27" layer="28" rot="MR180"/>
 </element>
@@
 </element>
 <element name="XTAL" library="murata-filter" package="CSTCE_V" value="CSTCE_V" x="19.3802" y="16.3068" smashed="yes" rot="R90"/>
-<element name="U$1" library="Logo" package="OSHW_10X500_NOTEXT" value="" x="20.0533" y="15.3416" smashed="yes" rot="MR0"/>
+<element name="U$1" library="Logo" package="OSHW_10X500_NOTEXT" value="" x="22.9743" y="14.3891" smashed="yes" rot="MR0"/>
 <element name="U1" library="Atmel_By_element14_Batch_1-00" package="QFP80P900X900X120-32N" value="ATMEGA328P-AU" x="11.5443" y="21.3614" smashed="yes" rot="R90">
 <attribute name="OC_FARNELL" value="1715486" x="11.5443" y="21.3614" size="1.778" layer="27" rot="R90" display="off"/>
@@
 </board>
 </drawing>
-<compatibility>
-<note version="6.3" minversion="6.2.2" severity="warning">
-Since Version 6.2.2 text objects can contain more than one line,
-which will not be processed correctly with this version.
-</note>
-</compatibility>
 </eagle>
