File: ApHSC.sch (EAGLE design)
At the start: 23 parts, among them U1 ATMEGA328P-AU, U2 UA78M05, U3 TPL7407L, U4 A2982

Commit message: Minor stylistic edits.
Other:
- note added: "ApHSC is an interface device designed to control an aftermarket heated seat control unit with a vehicle's stock control panel."
- note added: "Luis E Alvarado"
- note added: "https://goo.gl/t2CsID"
- moved on the sheet: C4, R5
Changed lines of the file:
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@@
 <setting verticaltext="up"/>
 </settings>
-<grid distance="0.1" unitdist="inch" unit="inch" style="lines" multiple="1" display="no" altdistance="0.01" altunitdist="inch" altunit="inch"/>
+<grid distance="0.5" unitdist="mm" unit="mm" style="lines" multiple="1" display="yes" altdistance="0.0025" altunitdist="inch" altunit="inch"/>
 <layers>
 <layer number="1" name="Top" color="4" fill="1" visible="no" active="no"/>
@@
 </layers>
 <schematic xreflabel="%F%N/%S.%C%R" xrefpart="/%S.%C%R">
-<description>&lt;a href=https://goo.gl/t2CsID&gt;&lt;b&gt;Arduino Power Heated Seat Controller&lt;/b&gt;&lt;/a&gt;</description>
+<description>&lt;h1&gt;&lt;a href=https://goo.gl/t2CsID&gt;&lt;b&gt;ApHSC&lt;/b&gt;&lt;/a&gt;&lt;/h1&gt;
+&lt;h2&gt;Arduino powered Heated Seats Controller&lt;/h2&gt;
+&lt;p&gt;&lt;a href=https://github.com/avluis/ApHSC&gt;Software&lt;/a&gt; |
+&lt;a href=https://github.com/avluis/ApHSC-Hardware&gt;Hardware&lt;/a&gt;&lt;p/&gt;</description>
 <attributes>
 </attributes>
@@
 <sheets>
 <sheet>
-<description>&lt;a href=https://goo.gl/t2CsID&gt;&lt;b&gt;Arduino Power Heated Seat Controller&lt;/b&gt;&lt;/a&gt;</description>
 <plain>
+<text x="217" y="20" size="2.54" layer="94" ratio="12">Luis E Alvarado</text>
+<text x="163" y="9" size="1.9304" layer="94" ratio="10">ApHSC is an interface device
+designed to control an
+aftermarket heated seat
+control unit with a vehicle's
+stock control panel.</text>
+<text x="163" y="4.881" size="2.54" layer="94" ratio="12">https://goo.gl/t2CsID</text>
 </plain>
 <instances>
@@
 <instance part="H-OUT" gate="G$1" x="220.98" y="66.04" rot="R180"/>
 <instance part="SUPPLY1" gate="GND" x="33.02" y="38.1"/>
-<instance part="R5" gate="G$1" x="104.14" y="93.98" rot="R270"/>
+<instance part="R5" gate="G$1" x="104.14" y="96.139" rot="R270"/>
 <instance part="SUPPLY2" gate="G$1" x="104.14" y="111.76"/>
-<instance part="C4" gate="G$1" x="35.56" y="109.22" rot="R270"/>
-<instance part="SUPPLY3" gate="G$1" x="43.18" y="111.76"/>
+<instance part="C4" gate="G$1" x="38.1" y="109.22" rot="R270"/>
+<instance part="SUPPLY3" gate="G$1" x="47.752" y="111.76"/>
 <instance part="SUPPLY4" gate="GND" x="27.94" y="106.68"/>
 <instance part="C3" gate="G$1" x="38.1" y="86.36" rot="R270"/>
@@
 <instance part="SUPPLY18" gate="GND" x="48.26" y="38.1"/>
 <instance part="U3" gate="G$1" x="170.18" y="106.68"/>
-<instance part="FRAME1" gate="G$1" x="0" y="0" smashed="yes">
-<attribute name="DRAWING_NAME" x="162.052" y="20.828" size="2.032" layer="94" font="vector"/>
-<attribute name="LAST_DATE_TIME" x="217.17" y="10.16" size="2.286" layer="94" font="vector"/>
-<attribute name="SHEET" x="230.505" y="5.08" size="2.54" layer="94" font="vector"/>
-</instance>
+<instance part="FRAME1" gate="G$1" x="0" y="0"/>
 <instance part="U4" gate="G$1" x="170.18" y="63.5"/>
 <instance part="SUPPLY5" gate="GND" x="154.94" y="91.44"/>
@@
 <pinref part="C4" gate="G$1" pin="2"/>
 <pinref part="SUPPLY4" gate="GND" pin="GND"/>
-<wire x1="27.94" y1="109.22" x2="30.48" y2="109.22" width="0.1524" layer="91"/>
+<wire x1="27.94" y1="109.22" x2="33.02" y2="109.22" width="0.1524" layer="91"/>
 </segment>
 <segment>
@@
 <segment>
 <pinref part="R5" gate="G$1" pin="2"/>
-<label x="100.584" y="91.186" size="1.778" layer="95" rot="R180"/>
 <pinref part="U1" gate="A" pin="PC6"/>
 <wire x1="88.9" y1="88.9" x2="104.14" y2="88.9" width="0.1524" layer="91"/>
+<wire x1="104.14" y1="88.9" x2="104.14" y2="91.059" width="0.1524" layer="91"/>
+<label x="104.394" y="88.8365" size="1.27" layer="95" ratio="12" xref="yes"/>
 </segment>
 <segment>
@@
 <pinref part="R5" gate="G$1" pin="1"/>
 <pinref part="SUPPLY2" gate="G$1" pin="VDD"/>
-<wire x1="104.14" y1="109.22" x2="104.14" y2="99.06" width="0.1524" layer="91"/>
+<wire x1="104.14" y1="109.22" x2="104.14" y2="101.219" width="0.1524" layer="91"/>
 </segment>
 <segment>
 <pinref part="C4" gate="G$1" pin="1"/>
 <pinref part="SUPPLY3" gate="G$1" pin="VDD"/>
-<wire x1="38.1" y1="109.22" x2="40.64" y2="109.22" width="0.1524" layer="91"/>
+<wire x1="40.64" y1="109.22" x2="43.688" y2="109.22" width="0.1524" layer="91"/>
 <pinref part="U1" gate="A" pin="AVCC"/>
-<wire x1="40.64" y1="109.22" x2="43.18" y2="109.22" width="0.1524" layer="91"/>
+<wire x1="43.688" y1="109.22" x2="47.752" y2="109.22" width="0.1524" layer="91"/>
 <wire x1="53.34" y1="99.06" x2="48.26" y2="99.06" width="0.1524" layer="91"/>
 <pinref part="U1" gate="A" pin="VCC"/>
@@
 <wire x1="48.26" y1="101.6" x2="48.26" y2="104.14" width="0.1524" layer="91"/>
 <junction x="48.26" y="101.6"/>
-<wire x1="48.26" y1="101.6" x2="40.64" y2="101.6" width="0.1524" layer="91"/>
-<wire x1="40.64" y1="101.6" x2="40.64" y2="109.22" width="0.1524" layer="91"/>
-<junction x="40.64" y="109.22"/>
+<wire x1="48.26" y1="101.6" x2="43.688" y2="101.6" width="0.1524" layer="91"/>
+<wire x1="43.688" y1="101.6" x2="43.688" y2="109.22" width="0.1524" layer="91"/>
+<junction x="43.688" y="109.22"/>
 </segment>
 <segment>
@@
 </schematic>
 </drawing>
+<compatibility>
+<note version="6.3" minversion="6.2.2" severity="warning">
+Since Version 6.2.2 text objects can contain more than one line,
+which will not be processed correctly with this version.
+</note>
+</compatibility>
 </eagle>
